File: kicad/pico_lta042b010f_carrier.kicad_pcb (KiCad board)
At the start: 2 copper layers, 100 x 52 mm, 32 parts, among them J1 LTA042B010F_FFC_36P_0.5mm, J2 USB-C 5V INPUT, J3 CCFL_INVERTER_13V8, U1 RaspberryPi_Pico_2W, U3 MC34063AD

Commit message: Correct D7 polarity in schematic and PCB artwork
Parts:
- moved D7 2.54 mm to (15.8, 33.8), turned to 90 degrees
Connections:
- D7 pad 1: -13V8 -> CPUMP_MID
- D7 pad 2: CPUMP_MID -> -13V8
Changed lines of the file:
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@@
 	(footprint "Diode_THT:D_DO-41_SOD81_P2.54mm_Vertical_KathodeUp"
 		(layer "F.Cu")
-		(at 15.75 31.25 -90)
+		(at 15.75 33.79 90)
 		(descr "Diode, DO-41_SOD81 series, Axial, Vertical, pin pitch=2.54mm, , length*diameter=5.2*2.7mm^2, , http://www.diodes.com/_files/packages/DO-41%20(Plastic).pdf")
 		(tags "Diode DO-41_SOD81 series Axial Vertical pin pitch 2.54mm  length 5.2mm diameter 2.7mm")
 		(property "Reference" "D7"
-			(at 5.111468 0 0)
+			(at -2.571468 0 0)
 			(layer "F.SilkS")
 			(effects
@@
 		)
 		(property "Datasheet" ""
-			(at 0 0 90)
+			(at 0 0 270)
 			(unlocked yes)
 			(layer "F.Fab")
@@
 		)
 		(property "Description" ""
-			(at 0 0 90)
+			(at 0 0 270)
 			(unlocked yes)
 			(layer "F.Fab")
@@
 		)
 		(fp_line
-			(start -1.35 1.6)
-			(end 4.15 1.6)
+			(start 4.15 -1.6)
+			(end -1.35 -1.6)
+			(stroke
+				(width 0.05)
+				(type solid)
+			)
+			(layer "F.CrtYd")
+		)
+		(fp_line
+			(start -1.35 -1.6)
+			(end -1.35 1.6)
 			(stroke
 				(width 0.05)
@@
 		)
 		(fp_line
-			(start -1.35 -1.6)
-			(end -1.35 1.6)
-			(stroke
-				(width 0.05)
-				(type solid)
-			)
-			(layer "F.CrtYd")
-		)
-		(fp_line
-			(start 4.15 -1.6)
-			(end -1.35 -1.6)
+			(start -1.35 1.6)
+			(end 4.15 1.6)
 			(stroke
 				(width 0.05)
@@
 		)
 		(pad "1" thru_hole rect
-			(at 0 0 90)
+			(at 0 0 270)
+			(size 2.2 2.2)
+			(drill 1.1)
+			(layers "*.Cu" "*.Mask")
+			(remove_unused_layers no)
+			(net 34 "CPUMP_MID")
+			(pinfunction "K")
+			(pintype "passive")
+		)
+		(pad "2" thru_hole oval
+			(at 2.54 0 270)
 			(size 2.2 2.2)
 			(drill 1.1)
@@
 			(remove_unused_layers no)
 			(net 4 "-13V8")
-			(pinfunction "K")
-			(pintype "passive")
-		)
-		(pad "2" thru_hole oval
-			(at 2.54 0 90)
-			(size 2.2 2.2)
-			(drill 1.1)
-			(layers "*.Cu" "*.Mask")
-			(remove_unused_layers no)
-			(net 34 "CPUMP_MID")
 			(pinfunction "A")
 			(pintype "passive")
