File: kicad/pico_lta042b010f_carrier.kicad_sch (KiCad schematic)
At the start: 23 parts, among them J1 LTA042B010F_FFC36, J2 USB-C 5V INPUT, J3 13V8 OUT, U1 RaspberryPi_Pico_2W, U3 MC34063AD

Commit message: Correct D7 polarity in schematic and PCB artwork
Connections:
- net -13V8: now also D7.2 (A); no longer D7.1 (K)
- net CPUMP_MID: now also D7.1 (K); no longer D7.2 (A)
Other:
- moved on the sheet: D7
Changed lines of the file:
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@@
 		(instances (project "pico_lta042b010f_carrier" (path "/10000000-0000-4000-8000-000000000001" (reference "C9") (unit 1))))
 	)
-(symbol (lib_id "Device:D_Schottky") (at 199.39 43.18 180) (unit 1)
+(symbol (lib_id "Device:D_Schottky") (at 199.39 43.18 0) (unit 1)
 		(exclude_from_sim no) (in_bom yes) (on_board yes) (dnp no)
 		(property "Reference" "D7" (at 199.39 38.1 0) (effects (font (size 1.27 1.27))))
